Commit message: add camera and optical links, camera sensor for gz

File: bme_gazebo_sensors/urdf/mogi_bot.urdf (robot description, URDF)
Before this commit: robot mogi_bot, 4 links, 3 joints
Links:
- added link camera_link, mass 0.1; collision box size=.05 .05 .05; visual box size=.05 .05 .05
- added link camera_link_optical
Joints:
- added joint camera_joint: type fixed, parent base_link, child camera_link, origin xyz=0.225 0 0.075 rpy=0 0 0, axis 0 1 0
- added joint camera_optical_joint: type fixed, parent camera_link, child camera_link_optical, origin xyz=0 0 0 rpy=-1.5707 0 -1.5707

Commit message: add simulated lidar to the robot

File: bme_gazebo_sensors/urdf/mogi_bot.urdf (robot description, URDF)
Before this commit: robot mogi_bot, 6 links, 5 joints
Links:
- added link scan_link, mass 1e-5; collision box size=.1 .1 .1; visual mesh filename=package://bme_gazebo_sensors/meshes/lidar.dae
Joints:
- added joint scan_joint: type fixed, parent base_link, child scan_link, origin xyz=0.0 0 0.15 rpy=0 0 0, axis 0 1 0

Commit message: add IMU

File: bme_gazebo_sensors/urdf/mogi_bot.urdf (robot description, URDF)
Before this commit: robot mogi_bot, 7 links, 6 joints
Links:
- added link imu_link
Joints:
- added joint imu_joint: type fixed, parent base_link, child imu_link, origin xyz=0 0 0 rpy=0 0 0

Commit message: fix camera related items in urdf

File: bme_gazebo_sensors/urdf/mogi_bot.urdf (robot description, URDF)
Before this commit: robot mogi_bot, 8 links, 7 joints
Links:
- link camera_link: geometry collision box size=.03 .03 .03; visual box size=.03 .03 .03

Commit message: add separate link and joint for GPS

File: bme_gazebo_sensors/urdf/mogi_bot.urdf (robot description, URDF)
Before this commit: robot mogi_bot, 8 links, 7 joints
Links:
- added link navsat_link
Joints:
- added joint navsat_joint: type fixed, parent base_link, child navsat_link, origin xyz=0 0 0 rpy=0 0 0

Commit message: create starter branch

File: bme_gazebo_sensors/urdf/mogi_bot.urdf (robot description, URDF)
Before this commit: robot mogi_bot, 9 links, 8 joints
Links:
- removed link camera_link
- removed link camera_link_optical
- removed link imu_link
- removed link navsat_link
- removed link scan_link
Joints:
- removed joint camera_joint
- removed joint camera_optical_joint
- removed joint imu_joint
- removed joint navsat_joint
- removed joint scan_joint
